Commit message: [FIX] update stl and urdf (the first link has center (0,0,0) now)

File: arm_description/urdf/xrb.urdf (robot description, URDF)
Before this commit: robot arm_description, 7 links, 6 joints
Links:
- link Link_6: mass 0.15 -> 0.19
Joints:
- joint Joint_1: origin xyz=-0.0214142437132751 0.0194456602348006 0.191605452072183 rpy=0.00211481861111635 0.0055702541140081 1.57079739593879 -> xyz=0.0 0.0 0.051 rpy=0.00211481861111635 0.0055702541140081 1.57079739593879
